File: 2021-2022 PCBs Complete/connector/CON_REVC.brd (EAGLE design)
At the start: 95.9 x 90.8 mm, 25 parts, among them J1 M80-5100642, J10 M80-5100642, J11 M80-5100642, J12 M80-5100642, J13 M80-5100642, J2 M80-5100642, J3 M80-5100642, J4 M80-5100642, J5 M80-5100642, J6 M80-5100642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

Commit message: JLCJLCJLC
Routing:
- net EMATCH2-: track 67.7 -> 69.7 mm
- net EMATCH1-: track 58.2 -> 60.2 mm
- net GND: vias 876 -> 873
Other:
- board text added: "JLCJLCJLC"
Changed lines of the file:
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@@
 <setting verticaltext="up"/>
 </settings>
-<grid distance="1" unitdist="mm" unit="mm" style="lines" multiple="1" display="yes" altdistance="1" altunitdist="mil" altunit="mil"/>
+<grid distance="5" unitdist="mm" unit="mm" style="lines" multiple="1" display="yes" altdistance="1" altunitdist="mil" altunit="mil"/>
 <layers>
-<layer number="1" name="Top" color="4" fill="1" visible="no" active="yes"/>
+<layer number="1" name="Top" color="4" fill="1" visible="yes" active="yes"/>
 <layer number="2" name="Route2" color="16" fill="1" visible="no" active="no"/>
 <layer number="3" name="Route3" color="17" fill="1" visible="no" active="no"/>
@@
 <layer number="14" name="Route14" color="22" fill="1" visible="no" active="no"/>
 <layer number="15" name="Route15" color="23" fill="1" visible="no" active="no"/>
-<layer number="16" name="Bottom" color="1" fill="1" visible="no" active="yes"/>
+<layer number="16" name="Bottom" color="1" fill="1" visible="yes" active="yes"/>
 <layer number="17" name="Pads" color="2" fill="1" visible="yes" active="yes"/>
-<layer number="18" name="Vias" color="2" fill="1" visible="no" active="yes"/>
-<layer number="19" name="Unrouted" color="6" fill="1" visible="no" active="yes"/>
-<layer number="20" name="Dimension" color="24" fill="1" visible="no" active="yes"/>
-<layer number="21" name="tPlace" color="7" fill="1" visible="no" active="yes"/>
+<layer number="18" name="Vias" color="2" fill="1" visible="yes" active="yes"/>
+<layer number="19" name="Unrouted" color="6" fill="1" visible="yes" active="yes"/>
+<layer number="20" name="Dimension" color="24" fill="1" visible="yes" active="yes"/>
+<layer number="21" name="tPlace" color="7" fill="1" visible="yes" active="yes"/>
 <layer number="22" name="bPlace" color="7" fill="1" visible="yes" active="yes"/>
-<layer number="23" name="tOrigins" color="15" fill="1" visible="no" active="yes"/>
-<layer number="24" name="bOrigins" color="15" fill="1" visible="no" active="yes"/>
-<layer number="25" name="tNames" color="7" fill="1" visible="no" active="yes"/>
-<layer number="26" name="bNames" color="7" fill="1" visible="no" active="yes"/>
+<layer number="23" name="tOrigins" color="15" fill="1" visible="yes" active="yes"/>
+<layer number="24" name="bOrigins" color="15" fill="1" visible="yes" active="yes"/>
+<layer number="25" name="tNames" color="7" fill="1" visible="yes" active="yes"/>
+<layer number="26" name="bNames" color="7" fill="1" visible="yes" active="yes"/>
 <layer number="27" name="tValues" color="7" fill="1" visible="no" active="yes"/>
 <layer number="28" name="bValues" color="7" fill="1" visible="no" active="yes"/>
@@
 <layer number="37" name="tTest" color="7" fill="1" visible="no" active="yes"/>
 <layer number="38" name="bTest" color="7" fill="1" visible="no" active="yes"/>
-<layer number="39" name="tKeepout" color="4" fill="11" visible="no" active="yes"/>
-<layer number="40" name="bKeepout" color="1" fill="11" visible="no" active="yes"/>
-<layer number="41" name="tRestrict" color="4" fill="10" visible="no" active="yes"/>
-<layer number="42" name="bRestrict" color="1" fill="10" visible="no" active="yes"/>
+<layer number="39" name="tKeepout" color="4" fill="11" visible="yes" active="yes"/>
+<layer number="40" name="bKeepout" color="1" fill="11" visible="yes" active="yes"/>
+<layer number="41" name="tRestrict" color="4" fill="10" visible="yes" active="yes"/>
+<layer number="42" name="bRestrict" color="1" fill="10" visible="yes" active="yes"/>
 <layer number="43" name="vRestrict" color="2" fill="10" visible="no" active="yes"/>
 <layer number="44" name="Drills" color="7" fill="1" visible="no" active="yes"/>
@@
 <layer number="49" name="Reference" color="7" fill="1" visible="no" active="yes"/>
 <layer number="50" name="dxf" color="7" fill="1" visible="no" active="no"/>
-<layer number="51" name="tDocu" color="7" fill="1" visible="no" active="yes"/>
-<layer number="52" name="bDocu" color="7" fill="1" visible="no" active="yes"/>
+<layer number="51" name="tDocu" color="7" fill="1" visible="yes" active="yes"/>
+<layer number="52" name="bDocu" color="7" fill="1" visible="yes" active="yes"/>
 <layer number="53" name="tGND_GNDA" color="7" fill="9" visible="no" active="no"/>
 <layer number="54" name="bGND_GNDA" color="1" fill="9" visible="no" active="no"/>
@@
 <text x="32.6136" y="83.3882" size="5" layer="22" rot="MR0">2</text>
 <text x="13.8176" y="83.2358" size="5" layer="22" rot="MR0">4</text>
+<text x="5.3302" y="60.0776" size="1.778" layer="21" rot="R90">JLCJLCJLC</text>
 </plain>
 <attributes>
@@
 <via x="7.9238" y="15.9238" extent="1-16" drill="0.35"/>
 <via x="8.9238" y="17.9238" extent="1-16" drill="0.35"/>
-<via x="7.9238" y="43.9238" extent="1-16" drill="0.35"/>
 <via x="8.9238" y="69.9238" extent="1-16" drill="0.35"/>
 <via x="7.9238" y="71.9238" extent="1-16" drill="0.35"/>
@@
 <via x="9.9238" y="15.9238" extent="1-16" drill="0.35"/>
 <via x="10.9238" y="17.9238" extent="1-16" drill="0.35"/>
-<via x="9.9238" y="43.9238" extent="1-16" drill="0.35"/>
 <via x="10.9238" y="69.9238" extent="1-16" drill="0.35"/>
 <via x="9.9238" y="71.9238" extent="1-16" drill="0.35"/>
@@
 <via x="12.9238" y="37.9238" extent="1-16" drill="0.35"/>
 <via x="12.9238" y="41.9238" extent="1-16" drill="0.35"/>
-<via x="11.9238" y="43.9238" extent="1-16" drill="0.35"/>
 <via x="12.9238" y="45.9238" extent="1-16" drill="0.35"/>
 <via x="12.9238" y="49.9238" extent="1-16" drill="0.35"/>
@@
 <wire x1="50" y1="48" x2="42" y2="48" width="2" layer="16"/>
 <wire x1="42" y1="48" x2="39" y2="45" width="2" layer="16"/>
+<wire x1="39" y1="43" x2="39" y2="41" width="1.524" layer="1"/>
 <wire x1="39" y1="43" x2="39" y2="41" width="2" layer="16"/>
 </signal>
@@
 <wire x1="39.0906" y1="50.8254" x2="35" y2="46.7348" width="2" layer="16"/>
 <wire x1="35" y1="43" x2="35" y2="41" width="2" layer="16"/>
+<wire x1="35" y1="43" x2="35" y2="41" width="1.524" layer="1"/>
 </signal>
 <signal name="EMATCH1_SUPPLY">
